File: PCB/page1.sch (EAGLE design)
At the start: 15 parts, among them IC3 MEGA16-A

Commit message: updated to version 3.2 of led PCB
Parts:
- removed IC3: MEGA16-A, atmel:MEGA16-A
- removed JP1: M05X2SHD_LOCK, SparkFun-Connectors:M05X2SHD_LOCK
- removed JP2: (no value), adafruit:PINHD-1X1
- removed LAMP: (no value), pinhead:PINHD-1X2
- removed MOTOR: (no value), pinhead-2:PINHD-1X06_2.00
- removed R1: 20k, rcl:R-US_R0805
- removed U$1: RJ-45-EDGE, Chris_parts:RJ-45-EDGE
- removed U$2: 742G04, Chris_parts:742G04
- removed U$3, U$4: N-FET_DUAL, Chris_parts:N-FET_DUAL
- added D1, D2, D3, D4, D5, D6, D7, D8: (no value), OPL Eagle Library:D-SMA
- added J1: RJ45-MJ88-BX11-RVSL2-3420050P1, OPL Eagle Library:RJ45-MJ88-BX11-RVSL2-3420050P1
- added J2: CONNECTOR-HEADER-6P-3460650P1, OPL Eagle Library:CONNECTOR-HEADER-6P-3460650P1
- added J4: CONNECTOR-HEADER-3P-3460810P1, OPL Eagle Library:CONNECTOR-HEADER-3P-3460810P1
- added J5: CONNECTOR-HEADER-2X3P-3460180P1, OPL Eagle Library:CONNECTOR-HEADER-2X3P-3460180P1
- added Q1, Q2, Q3, Q4: MOSFET-N-044020001, OPL Eagle Library:MOSFET-N-044020001
- added R3, R4: 10k, OPL Eagle Library:R-0603
- added U1: ATMEGA328P-AU-1030060P1, OPL Eagle Library:ATMEGA328P-AU-1030060P1
- added U2: L298-1420010P1, OPL Eagle Library:L298-1420010P1
- C1: value (none) -> 1uF; device rcl:C-USC2012 -> OPL Eagle Library:C-0805
- ISP: value (none) -> CONNECTOR-HEADER-2X3P-3460180P1; device pinhead:PINHD-2X3 -> OPL Eagle Library:CONNECTOR-HEADER-2X3P-3460180P1
- R2: value 20k -> 10k; device rcl:R-US_R0805 -> OPL Eagle Library:R-0603
Connections:
- removed net LED-: LAMP.2, U$1.3
- removed net N$2: U$2G$2.O, U$3G$2.G
- removed net N$6: MOTOR.1, U$4G$2.D
- removed net N$7: MOTOR.3, U$4G$1.D
- removed net N$8: MOTOR.4, U$3G$1.D
- removed net N$9: MOTOR.6, U$3G$2.D
- removed net TCK: IC3.(TCK)PC2, JP1.1
- removed net TDI: IC3.(TDI)PC5, JP1.9
- removed net TDO: IC3.(TDO)PC4, JP1.3
- removed net TMS: IC3.(TMS)PC3, JP1.5
- new net !A: Q1.D, R2.2, U2.IN2
- new net !B: Q2.D, R4.2, U2.IN3
- new net ENA: U2.ENA
- new net ENB: U2.ENB
- new net M1!A: D7.+, D8.-, J2.3, U2.OUT2
- new net M1!B: D3.+, D4.-, J2.5, J2.6, U2.OUT3
- new net M1A: D1.+, D2.-, J2.1, J2.2, U2.OUT1
- new net M1B: D5.+, D6.-, J2.4, U2.OUT4
- new net PB1: Q3.G, U1.PB1(OC1A)
- new net PB2: Q4.G, U1.PB2(SS/OC1B)
- net +12V: now also D1.-, D3.-, D5.-, D7.-, J1.8, J5.4, J5.5, J5.6, U2.VSS; no longer MOTOR.2, MOTOR.5, U$1.8
- net +5V: now also C1.2, ISP.6, J1.6, J1.G+, J4.2, R2.1, R4.1, U1.AREF, U1.AVCC, U1.VCC@1, U1.VCC@2, U2.VS; no longer C1.1, IC3.AREF, IC3.AVCC, IC3.VCC, IC3.VCC1, IC3.VCC2, ISP.2, JP1.4, LAMP.1, R1.2, U$1.6, U$2G$1.VCC
- net GND: now also C1.1, D2.+, D4.+, D6.+, D8.+, ISP.4, J1.7, J5.1, Q1.S, Q2.S, Q3.S, Q4.S, U1.GND, U1.GND@1, U1.GND@2, U2.GND@1, U2.GND@10, U2.GND@11, U2.GND@20, U2.SENSE_A, U2.SENSE_B, U2.THERMALS; no longer C1.2, IC3.GND, IC3.GND1, IC3.GND2, IC3.GND@1, ISP.6, JP1.10, JP1.2, U$1.7, U$2G$1.GND, U$3G$1.S, U$3G$2.S, U$4G$1.S, U$4G$2.S
- net LF1: now also U1.PD4(XCK/T0); no longer IC3.(T0/XCK)PB0
- net LF2: now also U1.PD5(T1); no longer IC3.(T1)PB1
- net MISO: now also U1.PB4(MISO); no longer IC3.(MISO)PB6
- net MOSI: now also ISP.5, R3.1; no longer IC3.(MOSI)PB5, ISP.4
- net N$1: now also J1.3, J4.1; no longer U$2G$3.O, U$4G$1.G
- net N$3: now also J5.3, Q4.D; no longer JP2.1, R2.2
- net N$4: now also J5.2, Q3.D; no longer IC3.(ADC4)PA4, IC3.(ADC5)PA5, IC3.(ADC6)PA6, IC3.(ADC7)PA7, R2.1
- net NC1: now also J1.2; no longer IC3.(OC1B)PD4, U$1.2
- net NC2: now also J1.5; no longer IC3.(INT1)PD3, U$1.5
- net OSC2A: now also Q1.G, R3.2, U1.PB3(MOSI/OC2), U2.IN1; no longer IC3.(ICP)PD6, U$2G$3.I, U$4G$2.G
- net OSC2B: now also Q2.G, U1.PD3(INT1), U2.IN4; no longer IC3.(OC2)PD7, U$2G$2.I, U$3G$1.G
- net RST: now also ISP.3, U1.PC6(/RESET); no longer IC3.RESET, ISP.5, JP1.6, R1.1
- net SCK: now also ISP.2, U1.PB5(SCK); no longer IC3.(SCK)PB7, ISP.3
- net S_RX: now also J1.4, U1.PD0(RXD); no longer IC3.(RXD)PD0, U$1.4
- net S_TX: now also J1.1, U1.PD1(TXD); no longer IC3.(TXD)PD1, U$1.1
Other:
- note removed: "actually mega164"

Commit message: Updated PCB design for ledboard 3.2r1
Connections:
- removed net ENA: U2.ENA
- removed net ENB: U2.ENB
- net +5V: now also U2.ENA, U2.ENB
Changed lines of the file:
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@@
 <part name="P+16" library="supply1" deviceset="+12V" device=""/>
 <part name="GND16" library="supply1" deviceset="GND" device=""/>
+<part name="P+17" library="supply1" deviceset="+5V" device=""/>
 </parts>
 <sheets>
@@
 <instance part="P+16" gate="1" x="358.14" y="106.68"/>
 <instance part="GND16" gate="1" x="317.5" y="91.44"/>
+<instance part="P+17" gate="1" x="297.18" y="27.94"/>
 </instances>
 <busses>
@@
 <wire x1="246.38" y1="22.86" x2="233.68" y2="22.86" width="0.1524" layer="91"/>
 <wire x1="233.68" y1="22.86" x2="233.68" y2="25.4" width="0.1524" layer="91"/>
+<pinref part="U2" gate="U" pin="ENA"/>
+<wire x1="246.38" y1="17.78" x2="231.14" y2="17.78" width="0.1524" layer="91"/>
+<wire x1="231.14" y1="17.78" x2="231.14" y2="22.86" width="0.1524" layer="91"/>
+<wire x1="231.14" y1="22.86" x2="233.68" y2="22.86" width="0.1524" layer="91"/>
+<junction x="233.68" y="22.86"/>
 </segment>
 <segment>
@@
 <pinref part="ISP" gate="J" pin="6"/>
 </segment>
+<segment>
+<pinref part="U2" gate="U" pin="ENB"/>
+<wire x1="276.86" y1="20.32" x2="297.18" y2="20.32" width="0.1524" layer="91"/>
+<pinref part="P+17" gate="1" pin="+5V"/>
+<wire x1="297.18" y1="20.32" x2="297.18" y2="25.4" width="0.1524" layer="91"/>
+</segment>
 </net>
 <net name="NC2" class="0">
@@
 </segment>
 </net>
-<net name="ENA" class="0">
-<segment>
-<pinref part="U2" gate="U" pin="ENA"/>
-<wire x1="246.38" y1="17.78" x2="233.68" y2="17.78" width="0.1524" layer="91"/>
-<label x="233.68" y="17.78" size="1.778" layer="95"/>
-</segment>
-</net>
-<net name="ENB" class="0">
-<segment>
-<pinref part="U2" gate="U" pin="ENB"/>
-<wire x1="276.86" y1="20.32" x2="292.1" y2="20.32" width="0.1524" layer="91"/>
-<label x="281.94" y="20.32" size="1.778" layer="95"/>
-</segment>
-</net>
