File: source/PCB/ODboard_3_5.kicad_pcb (KiCad board)
At the start: 2 copper layers, 74.9 x 45 mm, 18 parts, among them J1 RJ45, J3 CONN_01X04, J4 CONN_01X03, J5 CONN_02X03, Q3 CJ2302, Q4 CJ2302, U1 ATMEGA328P-A, U2 POLOLU_A4988

Commit message: update to kicad 5
Connections:
- J1 pad 2: Net-(J1-Pad2) -> (no net)
- J1 pad 5: Net-(J1-Pad5) -> (no net)
- U1 pad 19: Net-(U1-Pad19) -> (no net)
- U1 pad 22: Net-(U1-Pad22) -> (no net)
- U1 pad 26: Net-(U1-Pad26) -> (no net)
- U1 pad 27: Net-(U1-Pad27) -> (no net)
- U1 pad 28: Net-(U1-Pad28) -> (no net)
- U1 pad 7: Net-(U1-Pad7) -> (no net)
- U1 pad 8: Net-(U1-Pad8) -> (no net)
